File: Hardware/kiCAD/DataLogger.kicad_pcb (KiCad board)
At the start: 2 copper layers, 48.4 x 113.8 mm, 37 parts, among them J1 On/Off, J10 Conn_01x02_Pin, J2 RTC_Batt, J3 Uart1, J5 Mounting Hole, J6 Mounting Hole, J7 Mounting Hole, J8 Mounting Hole, Q1 2N7002, Q2 2N7002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

Commit message: TXS0104ED wiring fix and layout adjustments for improved SD card access. REV2.1
Parts:
- removed C2: 100n, Capacitor_SMD:C_0805_2012Metric_Pad1.18x1.45mm_HandSolder
- moved R7 29.0 mm to (144.6, 108.1), turned to -90 degrees
- moved SW2 27.3 mm to (147.3, 138.6)
- moved J1 26.1 mm to (157.6, 72.8)
- moved SW1 24.2 mm to (151.1, 113.3)
- moved C4 23.7 mm to (154.9, 95.1), turned to 90 degrees
- moved U2 23.3 mm to (149.4, 105.9), turned to 180 degrees
- moved Q1 22.9 mm to (127.3, 130.9)
- moved R8 22.9 mm to (126.5, 122.8)
- moved U3 22.9 mm to (154.7, 99.4), turned to -90 degrees
- moved C6 22.8 mm to (127.3, 127.1)
- moved R1 19.2 mm to (141.7, 116.9), turned to 90 degrees
- moved C3 19.0 mm to (151.9, 99.4), turned to -90 degrees
- moved R2 18.8 mm to (145.3, 116.9), turned to 90 degrees
- moved R3 18.1 mm to (148.9, 116.9), turned to 90 degrees
- moved R4 17.6 mm to (152.5, 116.9), turned to 90 degrees
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Connections:
- R7 pad 1: +1V8 -> +3V3
- T1 pad 0: Net-(U2-A1) -> Net-(U2-B2)
- T1 pad 1: Net-(U2-A2) -> Net-(U2-B1)
- T1 pad 14: Net-(U2-A3) -> Net-(U2-B3)
- U2 pad 1: +3V3 -> +1V8
- U2 pad 10: Net-(J3-Pin_6) -> Net-(U2-B3)
- U2 pad 11: Net-(J3-Pin_5) -> Net-(U2-B3)
- U2 pad 12: Net-(J3-Pin_4) -> Net-(U2-B2)
- U2 pad 13: Net-(J3-Pin_3) -> Net-(U2-B1)
- U2 pad 14: +1V8 -> +3V3
- U2 pad 2: Net-(U2-A1) -> Net-(J3-Pin_3)
- U2 pad 3: Net-(U2-A2) -> Net-(J3-Pin_4)
- U2 pad 4: Net-(U2-A3) -> Net-(J3-Pin_5)
- U2 pad 5: Net-(U2-A3) -> Net-(J3-Pin_6)
Routing:
- net Net-(J1-Pin_1): track 57.2 -> 128.1 mm
- net Net-(U2-B2): track 0.00 -> 37.1 mm
- net Net-(U1-LBO): track 82.7 -> 47.1 mm, vias 1 -> 2
- net Net-(U2-B1): track 0.00 -> 34.3 mm
- net Net-(BT1-+): track 46.3 -> 13.0 mm
- net Net-(U2-B3): track 0.00 -> 32.9 mm, vias 0 -> 1
- net Net-(U2-A2): track 30.1 -> 0.00 mm, vias 1 -> 0
- net Net-(U2-A1): track 27.1 -> 0.00 mm, vias 1 -> 0
- net +3V3: track 32.9 -> 58.3 mm, vias 3 -> 2
- net Net-(R4-Pad2): track 59.1 -> 34.5 mm
- net Net-(R3-Pad2): track 56.9 -> 33.0 mm
- net Net-(D1-K): track 14.0 -> 37.4 mm
- net Net-(R2-Pad2): track 55.4 -> 32.8 mm
- net Net-(R1-Pad2): track 53.7 -> 32.8 mm
- net +1V8: track 23.3 -> 3.79 mm
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Other:
- board size 48.4 x 113.8 mm -> 48.4 x 123.2 mm
- board text added: "Config.^"
- board text added: "West Lab Hydrophone Data Logger REV2.1"
- board text removed: "West Lab Hydrophone Data Logger REV2"
